Commit message: Updated

File: src/auv_slam/src/description/orca4_description.urdf (robot description, URDF)
Before this commit: robot orca4_ign, 10 links, 9 joints
Joints:
- joint thruster1_joint: axis 0 0 -1 -> 1 0 0; origin xyz=0.14 -0.092 0 rpy=-1.5707963267948966 1.5707963267948966 -0.7853981633974483 -> xyz=0.14 -0.092 0 rpy=0 0 -0.7853981633974483
- joint thruster2_joint: axis 0 0 -1 -> 1 0 0; origin xyz=0.14 0.092 0 rpy=-1.5707963267948966 1.5707963267948966 -2.356194490192345 -> xyz=0.14 0.092 0 rpy=0 0 -2.356194490192345
- joint thruster3_joint: axis 0 0 -1 -> 1 0 0; origin xyz=-0.14 -0.092 0 rpy=-1.5707963267948966 1.5707963267948966 0.7853981633974483 -> xyz=-0.14 -0.092 0 rpy=0 0 0.7853981633974483
- joint thruster4_joint: axis 0 0 -1 -> 1 0 0; origin xyz=-0.14 0.092 0 rpy=-1.5707963267948966 1.5707963267948966 2.356194490192345 -> xyz=-0.14 0.092 0 rpy=0 0 2.356194490192345
- joint thruster5_joint: axis 0 0 -1 -> 0 0 1
- joint thruster6_joint: axis 0 0 -1 -> 0 0 1

Commit message: Updated

File: src/auv_slam/src/description/orca4_description.urdf (robot description, URDF)
Before this commit: robot orca4_ign, 10 links, 9 joints
Links:
- added link camera_forward_link, mass 0.001; visual box 
Joints:
- added joint camera_forward_joint: type fixed, parent base_link, child camera_forward_link, origin xyz=0.23 0 0 rpy=0 0 0

Commit message: changed

File: src/auv_slam/src/description/orca4_description.urdf (robot description, URDF)
Before this commit: robot orca4_ign, 11 links, 10 joints
Links:
- removed link camera_forward_link
Joints:
- joint camera_forward_joint: origin xyz=0.23 0 0 rpy=0 0 0 -> xyz=0.23 0 0 rpy=0 0.2618 0

Commit message: Deleted Bt.py

File: src/auv_slam/src/description/orca4_description.urdf (robot description, URDF)
Before this commit: robot orca4_ign, 10 links, 10 joints
Links:
- added link camera_forward_link, mass 0.015; collision box size=0.03 0.06 0.03; visual box size=0.03 0.06 0.03

Commit message: Updated

File: src/auv_slam/src/description/orca4_description.urdf (robot description, URDF)
Before this commit: robot orca4_ign, 11 links, 10 joints
Joints:
- joint camera_forward_joint: origin xyz=0.23 0 0 rpy=0 0.2618 0 -> xyz=0.23 0 0 rpy=0 0 0

Commit message: Updated (bot spawned)

File: src/auv_slam/src/description/orca4_description.urdf (robot description, URDF)
Before this commit: robot orca4_ign, 11 links, 10 joints
Links:
- link imu_link: mass None -> 0.001; geometry collision box size=0.1 0.1 0.1; visual box size=0.1 0.1 0.1
Joints:
- joint imu_joint: origin xyz=0 0 0.01 -> xyz=0 0 0.01 rpy=0 0 0

Commit message: Removed qualification

File: src/auv_slam/src/description/orca4_description.urdf (robot description, URDF)
Before this commit: robot orca4_ign, 11 links, 10 joints
Links:
- link imu_link: mass 0.001 -> None; geometry collision box ; visual box 
Joints:
- joint imu_joint: origin xyz=0 0 0.01 rpy=0 0 0 -> xyz=0 0 0.01
